Commit message: fixed urdf for zed2

File: zed_wrapper/urdf/zed_macro.urdf.xacro (robot description, xacro)
@@ -45,5 +45,5 @@
       <xacro:property name="baseline" value="0.12" />
       <xacro:property name="height" value="0.03" />
-      <xacro:property name="bottom_slope" value="0.05" />
+      <xacro:property name="bottom_slope" value="0.0" />
       <xacro:property name="screw_offset_x" value="0.0" />
       <xacro:property name="screw_offset_z" value="0.0" />
